Commit message: Import .stl externally linked object, but the original grasp sampler is not working. Wait for fixing.

File: examples/pybullet/kuka/cook/models/mug.urdf (robot description, URDF)
Before this commit: robot mug, 1 links, 0 joints
Links:
- link LMS_link: geometry collision mesh filename=./stls/025_mug.stl scale=2.0; visual mesh filename=./stls/025_mug.stl scale=2.0

Commit message: Import .stl externally linked object, but the original grasp sampler is not working. Wait for fixing.

File: examples/pybullet/kuka/cook/models/mug.urdf (robot description, URDF)
Before this commit: robot mug, 1 links, 0 joints
Links:
- link LMS_link: geometry collision mesh filename=./stls/025_mug.obj scale=2.0; visual mesh filename=./stls/025_mug.obj scale=2.0
